Commit message: Create base robot chassis and RViz visualization

File: src/roborack_base/urdf/robot.xacro (robot description, xacro)
@@ -1,31 +1,6 @@
 <?xml version="1.0"?>
-<robot name="roborack" xmlns:xacro="http://www.ros.org/wiki/xacro">
-  <link name="base_link">
-    <visual>
-      <origin xyz="0 0 0.05"/>
-      <geometry>
-        <box size="0.40 0.30 0.10"/>
-      </geometry>
-      <material name="blue">
-        <color rgba="0.2 0.4 0.9 1"/>
-      </material>
-    </visual>
-    <collision>
-      <origin xyz="0 0 0.05"/>
-      <geometry>
-        <box size="0.40 0.30 0.10"/>
-      </geometry>
-    </collision>
-    <inertial>
-      <origin xyz="0 0 0.05"/>
-      <mass value="10.0"/>
-      <inertia
-        ixx="0.104"
-        ixy="0.0"
-        ixz="0.0"
-        iyy="0.167"
-        iyz="0.0"
-        izz="0.208"/>
-    </inertial>
-  </link>
+<robot name="roborack"
+       xmlns:xacro="http://www.ros.org/wiki/xacro">
+  <xacro:include filename="$(find roborack_base)/urdf/base.xacro"/>
+  <xacro:include filename="$(find roborack_base)/urdf/wheels.xacro"/>
 </robot>
