Commit message: Add base_footprint frame to robot model

File: src/roborack_base/urdf/base.xacro (robot description, xacro)
@@ -1,4 +1,10 @@
 <?xml version="1.0"?>
 <robot xmlns:xacro="http://www.ros.org/wiki/xacro">
+  <link name="base_footprint"/>
+  <joint name="base_footprint_joint" type="fixed">
+    <parent link="base_footprint"/>
+    <child link="base_link"/>
+    <origin xyz="0 0 0.05"/>
+</joint>
   <link name="base_link">
     <visual>

File: src/roborack_base/urdf/wheels.xacro (robot description, xacro)
@@ -1,10 +1,10 @@
 <?xml version="1.0"?>
 <robot xmlns:xacro="http://www.ros.org/wiki/xacro">
-  <!-- Left wheel -->
+  <!-- LEFT WHEEL -->
   <link name="left_wheel">
     <visual>
-      <origin xyz="0 0 0" rpy="1.5708 0 0"/>
+      <origin rpy="1.5708 0 0"/>
       <geometry>
-        <cylinder radius="0.05" length="0.03"/>
+        <cylinder radius="0.05" length="0.04"/>
       </geometry>
       <material name="black">
@@ -13,11 +13,11 @@
     </visual>
     <collision>
-      <origin xyz="0 0 0" rpy="1.5708 0 0"/>
+      <origin rpy="1.5708 0 0"/>
       <geometry>
-        <cylinder radius="0.05" length="0.03"/>
+        <cylinder radius="0.05" length="0.04"/>
       </geometry>
     </collision>
     <inertial>
-      <mass value="1.0"/>
+      <mass value="0.5"/>
       <inertia
         ixx="0.001"
@@ -29,21 +29,29 @@
     </inertial>
   </link>
-  <!-- Right wheel -->
+  <joint name="left_wheel_joint" type="continuous">
+    <parent link="base_link"/>
+    <child link="left_wheel"/>
+    <origin xyz="0 0.17 0.05"/>
+    <axis xyz="0 1 0"/>
+  </joint>
+  <!-- RIGHT WHEEL -->
   <link name="right_wheel">
     <visual>
-      <origin xyz="0 0 0" rpy="1.5708 0 0"/>
+      <origin rpy="1.5708 0 0"/>
       <geometry>
-        <cylinder radius="0.05" length="0.03"/>
+        <cylinder radius="0.05" length="0.04"/>
       </geometry>
-      <material name="black"/>
+      <material name="black">
+        <color rgba="0.1 0.1 0.1 1"/>
+      </material>
     </visual>
     <collision>
-      <origin xyz="0 0 0" rpy="1.5708 0 0"/>
+      <origin rpy="1.5708 0 0"/>
       <geometry>
-        <cylinder radius="0.05" length="0.03"/>
+        <cylinder radius="0.05" length="0.04"/>
       </geometry>
     </collision>
     <inertial>
-      <mass value="1.0"/>
+      <mass value="0.5"/>
       <inertia
         ixx="0.001"
@@ -55,16 +63,8 @@
     </inertial>
   </link>
-  <!-- Left wheel joint -->
-  <joint name="left_wheel_joint" type="continuous">
-    <parent link="base_link"/>
-    <child link="left_wheel"/>
-    <origin xyz="0 0.18 0.05"/>
-    <axis xyz="0 1 0"/>
-  </joint>
-  <!-- Right wheel joint -->
   <joint name="right_wheel_joint" type="continuous">
     <parent link="base_link"/>
     <child link="right_wheel"/>
-    <origin xyz="0 -0.18 0.05"/>
+    <origin xyz="0 -0.17 0.05"/>
     <axis xyz="0 1 0"/>
   </joint>
